File: loco-rollers-n.kicad_pcb (KiCad board)
At the start: 2 copper layers, 12.2 x 12.8 mm, 4 parts

Commit message: r1 pcb and gerbers
Parts:
- added G***: LOGO, loco-rollers-n:shinkansen_e5_mark_3000dpi_nocu, F.Cu at (156.9, 113.8)
Routing:
- net /PWR: track 0.00 -> 23.6 mm
- added copper zone on B.Cu, net /PWR
Other:
- net class Default: clearance 0.2 -> 0.254; trace_width 0.25 -> 0.508; via_dia 0.8 -> 0.6096; via_drill 0.4 -> 0.3048
- rule trace_clearance: 0.2 -> 0.254
- rule trace_min: 0.2 -> 0.1524
- board text added: "2020"
- board text added: "JLCJLCJLCJLC"
- board text added: "N Loco Rollers"
- board text added: "R1"
- board text added: "ihartwig"
- board text removed: "LocoRollers N"
- board text removed: "ihartwig P1 2020"
